File: Hardware/Buisness Card/Buisness Card.kicad_sch (KiCad schematic)
At the start: 25 parts, among them J101 USB_A, J102 Conn_01x03_Male, J103 Tag Connect, U101 NCP1117-12_SOT223, U102 ATtiny85-20S, U103 ProtoBoard

Commit message: Perform a lot of extra rework for a v.2
Parts:
- C103: value 4.7uf -> 5pf
- J103: footprint Connector:Tag-Connect_TC2050-IDC-NL_2x05_P1.27mm_Vertical -> Connector:Tag-Connect_TC2050-IDC-FP_2x05_P1.27mm_Vertical
Connections:
- net USB+: now also D102.1 (K), J101.3 (D+), R101.2, R103.1; no longer JP101.1 (A), R103.2, U102.2 (XTAL1/PB3)
- net USB-: now also D101.1 (K), J101.2 (D-), R102.1; no longer JP102.1 (A), R102.2, U102.3 (XTAL2/PB4)
- new net USBA: JP101.1 (A), R103.2, U102.2 (XTAL1/PB3)
- new net USBB: JP102.1 (A), R102.2, U102.3 (XTAL2/PB4)
Other:
- note removed: "Ask dad if this is ok setup"
- moved on the sheet: C101, J102
