File: Hardware/Buisness Card/Buisness Card.kicad_pcb (KiCad board)
At the start: 2 copper layers, 100.7 x 62.9 mm, 35 parts, among them J101 USB_A, J102 Conn_01x03_Male, J103 Tag Connect, P1 USB_A, U101 NCP1117-12_SOT223, U102 ATtiny85-20S, U103 ProtoBoard

Commit message: Start to make changes for a sleeker design
Parts:
- moved U103 12.7 mm to (159.0, 101.6)
Routing:
- net (no net): track 106.7 -> 81.3 mm
- net +5V: track 278.1 -> 279.4 mm
- net /SDO: track 61.1 -> 61.9 mm

Commit message: Perform a lot of extra rework for a v.2
Parts:
- C103: value 4.7uf -> 5pf
- J103: footprint Connector:Tag-Connect_TC2050-IDC-NL_2x05_P1.27mm_Vertical -> Connector:Tag-Connect_TC2050-IDC-FP_2x05_P1.27mm_Vertical
- moved J103 46.8 mm to (171.5, 82.0), turned to 45 degrees
- moved C102 13.5 mm to (175.8, 103.9), turned to -135 degrees
- moved U101 13.2 mm to (172.5, 99.6), turned to 135 degrees
- moved J102 13.2 mm to (164.8, 125.2)
- moved C101 11.0 mm to (178.8, 100.8), turned to 45 degrees
- moved R105 8.27 mm to (175.7, 90.0), turned to 45 degrees
- moved D102 7.47 mm to (186.9, 92.7)
- moved C103 7.47 mm to (180.6, 96.8)
- moved D105 7.47 mm to (184.7, 96.0)
- moved JP101 7.47 mm to (177.3, 87.4)
- moved JP102 7.47 mm to (179.1, 85.6)
- moved R101 7.47 mm to (187.2, 89.9)
- moved R102 7.47 mm to (183.6, 86.6)
- moved R103 7.47 mm to (185.0, 88.0)
- moved U102 7.47 mm to (179.8, 91.7)
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Connections:
- D101 pad 1: Net-(D101-Pad1) -> /USB-
- D102 pad 1: Net-(D102-Pad1) -> /USB+
- J101 pad 2: Net-(D101-Pad1) -> /USB-
- J101 pad 3: Net-(D102-Pad1) -> /USB+
- JP101 pad 1: /USB+ -> /USBA
- JP102 pad 1: /USB- -> /USBB
- R101 pad 2: Net-(D102-Pad1) -> /USB+
- R102 pad 1: Net-(D101-Pad1) -> /USB-
- R102 pad 2: /USB- -> /USBB
- R103 pad 1: Net-(D102-Pad1) -> /USB+
- R103 pad 2: /USB+ -> /USBA
- U102 pad 2: /USB+ -> /USBA
- U102 pad 3: /USB- -> /USBB
Routing:
- net (no net): track 81.3 -> 0.00 mm, vias 4 -> 0
- net +5V: track 279.4 -> 232.3 mm, vias 7 -> 4
- net /SDI: track 63.2 -> 25.6 mm, vias 2 -> 1
- net /SDO: track 61.9 -> 25.5 mm, vias 3 -> 0
- net /SCK: track 43.6 -> 27.8 mm, vias 3 -> 1
- net Net-(D102-Pad1): track 13.9 -> 0.00 mm
- net Net-(D101-Pad1): track 10.8 -> 0.00 mm
- net /USB+: track 8.43 -> 18.1 mm
- net Net-(D105-Pad2): track 29.6 -> 20.8 mm
- net /USBA: track 0.00 -> 8.22 mm
- net /USBB: track 0.00 -> 7.70 mm
- net /USB-: track 7.72 -> 15.1 mm
- net Net-(C101-Pad1): track 24.5 -> 29.5 mm
- net Net-(JP102-Pad2): track 22.6 -> 26.8 mm
- net Net-(D104-Pad1): track 5.36 -> 9.15 mm, vias 0 -> 2
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Other:
- board text added: "Find instructions on how to use with this QR code!"
- board text added: "Kitsune Scientific ${EMAIL} ${WEBSITE} ${PHONE}"
- board text added: "VIN"
- board text removed: "5V"
- board text removed: "Find instructions on how to use with the QR code above!"
- board text removed: "Kitsune Scientific ${EMAIL} ${DISCORD} ${WEBSITE} ${CALLSIGN}"

Commit message: Include revision tag next to jlc number
Other:
- board text added: "${REVISION}"
Changed lines of the file:
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@@
     )
   )
-  (property "FULL_REVISION" "v1.0-2-gf87380a")
-  (property "ISSUE" "2022-10-04")
+  (property "CALLSIGN" "Y0UR")
+  (property "EMAIL" "YourEmail@email.com")
+  (property "FULL_REVISION" "v1.0-3-g16be60e")
+  (property "ISSUE" "2022-10-07")
   (property "KENWOODFOX_3DMODELS" "Hardware/Buisness Card/Libraries/kenwoodfox-kicad-libraries/3d")
+  (property "NAME" "Your Name")
+  (property "PHONE" "+X(XXX)XXX-XXXX")
+  (property "REVISION" "16be60e")
+  (property "WEBSITE" "https://YourWebsite.net/")
   (net 0 "")
   (net 1 "/SDO")
@@
   (gr_arc (start 202.146 83.946) (mid 202.1528 80.4604) (end 205.6384 80.4672) (layer "Edge.Cuts") (width 0.1))
   (gr_line (start 114.3 123.19) (end 114.3 80.01) (layer "Edge.Cuts") (width 0.1))
-  (gr_text "JLCJLCJLCJLC" (at 117.094 121.158 -90) (layer "B.SilkS")
-    (effects (font (size 0.85 0.85) (thickness 0.2)) (justify left mirror))
+  (gr_text "${REVISION}" (at 116.078 121.158 -90) (layer "B.SilkS")
+    (effects (font (size 0.9 0.9) (thickness 0.2)) (justify left mirror))
+  )
+  (gr_text "JLCJLCJLCJLC" (at 118.11 121.158 -90) (layer "B.SilkS")
+    (effects (font (size 0.9 0.9) (thickness 0.2)) (justify left mirror))
   )
   (gr_text "Find instructions on how to use\nwith this QR code!" (at 186.944 91.186 315) (layer "B.SilkS")

Commit message: Bump and make curvy
Routing:
- net +5V: track 232.3 -> 227.6 mm
- net /USB+: track 18.1 -> 15.0 mm
- net /SDI: track 25.6 -> 24.0 mm
- net /SCK: track 27.8 -> 26.2 mm
- net /USB-: track 15.1 -> 13.5 mm
- net GND: track 7.97 -> 9.36 mm
- net /SDO: track 25.5 -> 24.1 mm
- net Net-(C101-Pad1): track 29.5 -> 28.3 mm
- net /RST: track 46.7 -> 45.6 mm

Commit message: Prep for new order
Routing:
- net /SDO: track 24.1 -> 22.7 mm
