File: Hardware/Buisness Card/Buisness Card.kicad_pcb (KiCad board)
At the start: 2 copper layers, 100.7 x 62.9 mm, 35 parts, among them J101 USB_A, J102 Conn_01x03_Male, J103 Tag Connect, P1 USB_A, U101 NCP1117-12_SOT223, U102 ATtiny85-20S, U103 ProtoBoard

Commit message: V2.0 Design (#1)
Parts:
- C103: value 4.7uf -> 5pf
- J103: footprint Connector:Tag-Connect_TC2050-IDC-NL_2x05_P1.27mm_Vertical -> Connector:Tag-Connect_TC2050-IDC-FP_2x05_P1.27mm_Vertical
- moved J103 46.8 mm to (171.5, 82.0), turned to 45 degrees
- moved C102 13.5 mm to (175.8, 103.9), turned to -135 degrees
- moved U101 13.2 mm to (172.5, 99.6), turned to 135 degrees
- moved J102 13.2 mm to (164.8, 125.2)
- moved U103 12.7 mm to (159.0, 101.6)
- moved C101 11.0 mm to (178.8, 100.8), turned to 45 degrees
- moved R105 8.27 mm to (175.7, 90.0), turned to 45 degrees
- moved D102 7.47 mm to (186.9, 92.7)
- moved C103 7.47 mm to (180.6, 96.8)
- moved D105 7.47 mm to (184.7, 96.0)
- moved JP101 7.47 mm to (177.3, 87.4)
- moved JP102 7.47 mm to (179.1, 85.6)
- moved R101 7.47 mm to (187.2, 89.9)
- moved R102 7.47 mm to (183.6, 86.6)
- moved R103 7.47 mm to (185.0, 88.0)
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Connections:
- D101 pad 1: Net-(D101-Pad1) -> /USB-
- D102 pad 1: Net-(D102-Pad1) -> /USB+
- J101 pad 2: Net-(D101-Pad1) -> /USB-
- J101 pad 3: Net-(D102-Pad1) -> /USB+
- JP101 pad 1: /USB+ -> /USBA
- JP102 pad 1: /USB- -> /USBB
- R101 pad 2: Net-(D102-Pad1) -> /USB+
- R102 pad 1: Net-(D101-Pad1) -> /USB-
- R102 pad 2: /USB- -> /USBB
- R103 pad 1: Net-(D102-Pad1) -> /USB+
- R103 pad 2: /USB+ -> /USBA
- U102 pad 2: /USB+ -> /USBA
- U102 pad 3: /USB- -> /USBB
Routing:
- net (no net): track 106.7 -> 0.00 mm, vias 4 -> 0
- net +5V: track 278.1 -> 227.6 mm, vias 7 -> 4
- net /SDI: track 63.2 -> 24.0 mm, vias 2 -> 1
- net /SDO: track 61.1 -> 22.7 mm, vias 3 -> 0
- net /SCK: track 43.6 -> 26.2 mm, vias 3 -> 1
- net Net-(D102-Pad1): track 13.9 -> 0.00 mm
- net Net-(D101-Pad1): track 10.8 -> 0.00 mm
- net Net-(D105-Pad2): track 29.6 -> 20.6 mm
- net /USBA: track 0.00 -> 7.86 mm
- net /USBB: track 0.00 -> 7.77 mm
- net /USB+: track 8.43 -> 15.0 mm
- net /USB-: track 7.72 -> 13.6 mm
- net GND: track 5.40 -> 9.35 mm, vias 4 -> 5
- net Net-(C101-Pad1): track 24.5 -> 28.3 mm
- net Net-(JP102-Pad2): track 22.6 -> 26.4 mm
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Other:
- board text added: "${REVISION}"
- board text added: "Find instructions on how to use with this QR code!"
- board text added: "Kitsune Scientific ${EMAIL} ${WEBSITE} ${PHONE}"
- board text added: "VIN"
- board text removed: "5V"
- board text removed: "Find instructions on how to use with the QR code above!"
- board text removed: "Kitsune Scientific ${EMAIL} ${DISCORD} ${WEBSITE} ${CALLSIGN}"
